File: CR2032 emulator.brd (EAGLE design)
At the start: 20 x 57 mm, 16 parts, among them CON1 USB_PWR-31-M-17, CON2 PINHEAD_1X02-2, IC2 RY6050-ADJM5R, SW1 SPDT_SWITCH

Commit message: attribute updates
Parts:
- R3: value 24K -> 2K
Changed lines of the file:
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@@
 </layers>
 <board>
-<fusionsync huburn="a.cGVyc29uYWw6dWUyYWE4ZDY4" projecturn="a.cGVyc29uYWw6dWUyYWE4ZDY4IzIwMTkwOTA2MjEzMTk3ODU2" f3durn="urn:adsk.wipprod:dm.lineage:Xbatf6oeTpqPrVNiO6yIyA" pcbguid="" lastpulledtime="" lastsyncedchangeguid="" latestrevisionid="49c072a4-3f1f-4bd7-ab2a-1c5ebe951bb5" lastsyncedrevisionid="49c072a4-3f1f-4bd7-ab2a-1c5ebe951bb5" lastboardhashguid="79a36a56-b72d-02e6-0152-9a1d112cce1a" lastpushedtime="2022-04-07T11:57:16Z" linktopcb3d="true"/>
+<fusionsync huburn="a.cGVyc29uYWw6dWUyYWE4ZDY4" projecturn="a.cGVyc29uYWw6dWUyYWE4ZDY4IzIwMTkwOTA2MjEzMTk3ODU2" f3durn="urn:adsk.wipprod:dm.lineage:Xbatf6oeTpqPrVNiO6yIyA" pcbguid="" lastpulledtime="" lastsyncedchangeguid="" latestrevisionid="31a8649d-6013-4b3f-8fdb-d08e69e8f611" lastsyncedrevisionid="31a8649d-6013-4b3f-8fdb-d08e69e8f611" lastboardhashguid="3ea0b9cb-6f79-6d17-c5f0-c3754e4f6761" lastpushedtime="2022-04-07T12:02:38Z" linktopcb3d="true"/>
 <plain>
 <circle x="0" y="0" radius="10" width="0.01" layer="51"/>
@@
 </attributes>
 <variantdefs>
+<variantdef name="basic" current="yes"/>
 </variantdefs>
 <classes>
@@
 <element name="R1" library="rc" library_urn="urn:adsk.eagle:library:2539423" package="R0603" package3d_urn="urn:adsk.eagle:package:2539454/2" value="100K" x="-1.4" y="-16.1" smashed="yes" rot="R180">
 <attribute name="AEC-Q" value="" x="-1.4" y="-16.1" size="1.778" layer="27" rot="R180" display="off"/>
-<attribute name="ALLOCATED" value="" x="-1.4" y="-16.1" size="1.778" layer="27" rot="R180" display="off"/>
+<attribute name="ALLOCATED" value="+" x="-1.4" y="-16.1" size="1.778" layer="27" rot="R180" display="off"/>
 <attribute name="DIGIKEY#" value="" x="-1.4" y="-16.1" size="1.778" layer="27" rot="R180" display="off"/>
-<attribute name="LCSC#" value="" x="-1.4" y="-16.1" size="1.778" layer="27" rot="R180" display="off"/>
+<attribute name="LCSC#" value="C25803" x="-1.4" y="-16.1" size="1.778" layer="27" rot="R180" display="off"/>
 <attribute name="MANF" value="" x="-1.4" y="-16.1" size="1.778" layer="27" rot="R180" display="off"/>
 <attribute name="MANF#" value="" x="-1.4" y="-16.1" size="1.778" layer="27" rot="R180" display="off"/>
@@
 <element name="R2" library="rc" library_urn="urn:adsk.eagle:library:2539423" package="R0603" package3d_urn="urn:adsk.eagle:package:2539454/2" value="24K" x="0.8" y="-20.1" smashed="yes" rot="R90">
 <attribute name="AEC-Q" value="" x="0.8" y="-20.1" size="1.778" layer="27" rot="R90" display="off"/>
-<attribute name="ALLOCATED" value="" x="0.8" y="-20.1" size="1.778" layer="27" rot="R90" display="off"/>
+<attribute name="ALLOCATED" value="+" x="0.8" y="-20.1" size="1.778" layer="27" rot="R90" display="off"/>
 <attribute name="DIGIKEY#" value="" x="0.8" y="-20.1" size="1.778" layer="27" rot="R90" display="off"/>
-<attribute name="LCSC#" value="" x="0.8" y="-20.1" size="1.778" layer="27" rot="R90" display="off"/>
+<attribute name="LCSC#" value="C23352" x="0.8" y="-20.1" size="1.778" layer="27" rot="R90" display="off"/>
 <attribute name="MANF" value="" x="0.8" y="-20.1" size="1.778" layer="27" rot="R90" display="off"/>
 <attribute name="MANF#" value="" x="0.8" y="-20.1" size="1.778" layer="27" rot="R90" display="off"/>
@@
 <element name="R2_" library="rc" library_urn="urn:adsk.eagle:library:2539423" package="R0603" package3d_urn="urn:adsk.eagle:package:2539454/2" value="36K" x="-1.4" y="-13.5" smashed="yes">
 <attribute name="AEC-Q" value="" x="-1.4" y="-13.5" size="1.778" layer="27" display="off"/>
-<attribute name="ALLOCATED" value="" x="-1.4" y="-13.5" size="1.778" layer="27" display="off"/>
+<attribute name="ALLOCATED" value="+" x="-1.4" y="-13.5" size="1.778" layer="27" display="off"/>
 <attribute name="DIGIKEY#" value="" x="-1.4" y="-13.5" size="1.778" layer="27" display="off"/>
-<attribute name="LCSC#" value="" x="-1.4" y="-13.5" size="1.778" layer="27" display="off"/>
+<attribute name="LCSC#" value="C23147" x="-1.4" y="-13.5" size="1.778" layer="27" display="off"/>
 <attribute name="MANF" value="" x="-1.4" y="-13.5" size="1.778" layer="27" display="off"/>
 <attribute name="MANF#" value="" x="-1.4" y="-13.5" size="1.778" layer="27" display="off"/>
@@
 <attribute name="VOLTAGE" value="" x="-1.4" y="-17.4" size="1.778" layer="27" rot="R180" display="off"/>
 </element>
-<element name="CON2" library="pinhead" library_urn="urn:adsk.eagle:library:2540341" package="1X02-PTH-2" package3d_urn="urn:adsk.eagle:package:6503394/4" value="PINHEAD_1X02-2" x="-4.1" y="-13" smashed="yes" rot="R270"/>
-<element name="R3" library="rc" library_urn="urn:adsk.eagle:library:2539423" package="R0603" package3d_urn="urn:adsk.eagle:package:2539454/2" value="24K" x="-1.4" y="-12.2" smashed="yes" rot="R180">
+<element name="CON2" library="pinhead" library_urn="urn:adsk.eagle:library:2540341" package="1X02-PTH-2" package3d_urn="urn:adsk.eagle:package:6503394/4" value="PINHEAD_1X02-2" x="-4.1" y="-13" populate="no" smashed="yes" rot="R270"/>
+<element name="R3" library="rc" library_urn="urn:adsk.eagle:library:2539423" package="R0603" package3d_urn="urn:adsk.eagle:package:2539454/2" value="2K" x="-1.4" y="-12.2" smashed="yes" rot="R180">
 <attribute name="AEC-Q" value="" x="-1.4" y="-12.2" size="1.778" layer="27" rot="R180" display="off"/>
-<attribute name="ALLOCATED" value="" x="-1.4" y="-12.2" size="1.778" layer="27" rot="R180" display="off"/>
+<attribute name="ALLOCATED" value="+" x="-1.4" y="-12.2" size="1.778" layer="27" rot="R180" display="off"/>
 <attribute name="DIGIKEY#" value="" x="-1.4" y="-12.2" size="1.778" layer="27" rot="R180" display="off"/>
-<attribute name="LCSC#" value="" x="-1.4" y="-12.2" size="1.778" layer="27" rot="R180" display="off"/>
+<attribute name="LCSC#" value="C22975" x="-1.4" y="-12.2" size="1.778" layer="27" rot="R180" display="off"/>
 <attribute name="MANF" value="" x="-1.4" y="-12.2" size="1.778" layer="27" rot="R180" display="off"/>
 <attribute name="MANF#" value="" x="-1.4" y="-12.2" size="1.778" layer="27" rot="R180" display="off"/>
@@
 </element>
 <element name="LED1" library="rc" library_urn="urn:adsk.eagle:library:2539423" package="LED0603" package3d_urn="urn:adsk.eagle:package:2539471/4" value="LED-0603" x="-1.4" y="-14.8" smashed="yes" rot="R180">
-<attribute name="COLOR" value="" x="-1.4" y="-14.8" size="1.778" layer="27" rot="R180" display="off"/>
+<attribute name="COLOR" value="Emerald" x="-1.4" y="-14.8" size="1.778" layer="27" rot="R180" display="off"/>
 <attribute name="DIGIKEY#" value="" x="-1.4" y="-14.8" size="1.778" layer="27" rot="R180" display="off"/>
-<attribute name="LCSC#" value="" x="-1.4" y="-14.8" size="1.778" layer="27" rot="R180" display="off"/>
+<attribute name="LCSC#" value="C72043" x="-1.4" y="-14.8" size="1.778" layer="27" rot="R180" display="off"/>
 <attribute name="MANF" value="" x="-1.4" y="-14.8" size="1.778" layer="27" rot="R180" display="off"/>
 <attribute name="MANF#" value="" x="-1.4" y="-14.8" size="1.778" layer="27" rot="R180" display="off"/>
@@
 <attribute name="VALUE" x="-1.4" y="-15.8" size="0.5" layer="27" font="vector" ratio="15" rot="R180" align="center"/>
 </element>
-<element name="SJ1" library="misc" library_urn="urn:adsk.eagle:library:5347860" package="SOLDER_JOINT_SMALL" package3d_urn="urn:adsk.eagle:package:35137462/1" value="" x="-4.1" y="-13" smashed="yes" rot="R90">
+<element name="SJ1" library="misc" library_urn="urn:adsk.eagle:library:5347860" package="SOLDER_JOINT_SMALL" package3d_urn="urn:adsk.eagle:package:35137462/1" value="" x="-4.1" y="-13" populate="no" smashed="yes" rot="R90">
 <attribute name="NAME" x="-5.6" y="-13" size="1" layer="25" font="vector" ratio="15" rot="R90" align="center"/>
 </element>
-<element name="PAD1" library="PADS" library_urn="urn:adsk.eagle:library:3188696" package="3X1.5" package3d_urn="urn:adsk.eagle:package:4854322/2" value="PAD-3X1.5" x="0" y="-7" smashed="yes">
+<element name="PAD1" library="PADS" library_urn="urn:adsk.eagle:library:3188696" package="3X1.5" package3d_urn="urn:adsk.eagle:package:4854322/2" value="PAD-3X1.5" x="0" y="-7" populate="no" smashed="yes">
 <attribute name="BOM" value="EXCLUDE" x="0" y="-7" size="1.778" layer="27" display="off"/>
 <attribute name="NAME" x="0" y="-7" size="1.27" layer="25" font="vector" ratio="15" align="center"/>
 </element>
-<element name="PAD2" library="PADS" library_urn="urn:adsk.eagle:library:3188696" package="HOLE_0.6" package3d_urn="urn:adsk.eagle:package:6513718/2" value="PAD-HOLE-0.6" x="-1" y="11" smashed="yes" rot="R90">
+<element name="PAD2" library="PADS" library_urn="urn:adsk.eagle:library:3188696" package="HOLE_0.6" package3d_urn="urn:adsk.eagle:package:6513718/2" value="PAD-HOLE-0.6" x="-1" y="11" populate="no" smashed="yes" rot="R90">
 <attribute name="NAME" x="-1" y="12" size="1.27" layer="25" font="vector" ratio="15" rot="R90" align="center-left"/>
 </element>
-<element name="PAD3" library="PADS" library_urn="urn:adsk.eagle:library:3188696" package="HOLE_0.6" package3d_urn="urn:adsk.eagle:package:6513718/2" value="PAD-HOLE-0.6" x="0" y="11" smashed="yes" rot="R90">
+<element name="PAD3" library="PADS" library_urn="urn:adsk.eagle:library:3188696" package="HOLE_0.6" package3d_urn="urn:adsk.eagle:package:6513718/2" value="PAD-HOLE-0.6" x="0" y="11" populate="no" smashed="yes" rot="R90">
 <attribute name="NAME" x="0" y="12" size="1.27" layer="25" font="vector" ratio="15" rot="R90" align="center-left"/>
 </element>
-<element name="PAD4" library="PADS" library_urn="urn:adsk.eagle:library:3188696" package="HOLE_0.6" package3d_urn="urn:adsk.eagle:package:6513718/2" value="PAD-HOLE-0.6" x="1" y="11" smashed="yes" rot="R90">
+<element name="PAD4" library="PADS" library_urn="urn:adsk.eagle:library:3188696" package="HOLE_0.6" package3d_urn="urn:adsk.eagle:package:6513718/2" value="PAD-HOLE-0.6" x="1" y="11" populate="no" smashed="yes" rot="R90">
 <attribute name="NAME" x="1" y="12" size="1.27" layer="25" font="vector" ratio="15" rot="R90" align="center-left"/>
 </element>
